File: pcb/pcb.kicad_pcb (KiCad board)
At the start: 2 copper layers, 284.6 x 110.1 mm, 149 parts, among them J1 USB_C_Receptacle_USB2.0, J2 USB_C_Receptacle_USB2.0, J4 USB_C_Receptacle_USB2.0, J5 USB_C_Receptacle_USB2.0, J6 PGA2040, SW3 RESET, SW4 BOOTSEL, U1 SL2.1A

Commit message: curved pcb
Routing:
- net /D4-: track 225.0 -> 223.4 mm
- net col11: track 340.3 -> 338.8 mm
- net col12: track 330.4 -> 329.2 mm
- net col13: track 309.2 -> 308.3 mm
Other:
- outline, holes or cut-outs redrawn

Commit message: Added Mounting Holes
Parts:
- added REF**: MountingHole_2.1mm, MountingHole:MountingHole_2.1mm, F.Cu at (228.1, 109.4)
- added REF**: MountingHole_2.1mm, MountingHole:MountingHole_2.1mm, F.Cu at (88.8, 108.8)
- added REF**: MountingHole_2.1mm, MountingHole:MountingHole_2.1mm, F.Cu at (231.7, 207.0)
- added REF**: MountingHole_2.1mm, MountingHole:MountingHole_2.1mm, F.Cu at (365.0, 109.4)
- added REF**: MountingHole_2.1mm, MountingHole:MountingHole_2.1mm, F.Cu at (88.8, 211.8)
- added REF**: MountingHole_2.1mm, MountingHole:MountingHole_2.1mm, F.Cu at (365.6, 211.8)
Routing:
- net col8: track 391.0 -> 387.9 mm
- net col9: track 378.0 -> 375.0 mm
- net col10: track 359.1 -> 356.4 mm
- net Net-(J1-CC2): track 22.1 -> 19.5 mm
- net /D4-: track 223.4 -> 222.7 mm
