File: pcb/pcb.kicad_pcb (KiCad board)
At the start: 2 copper layers, 284.6 x 110.1 mm, 155 parts, among them J1 USB_C_Receptacle_USB2.0, J2 USB_C_Receptacle_USB2.0, J4 USB_C_Receptacle_USB2.0, J5 USB_C_Receptacle_USB2.0, J6 PGA2040, SW3 RESET, SW4 BOOTSEL, U1 SL2.1A

Commit message: Added Proper Support
Parts:
- removed the REF** at (103.0, 144.5)
- removed the REF** at (341.1, 182.6)
- removed the REF** at (348.3, 163.5)
- removed the REF** at (214.9, 201.6)
- removed the REF** at (103.0, 163.5)
- removed the REF** at (350.6, 125.4)
- added REF**: Stabilizer_MX_6.25u, ScottoKeebs_Stabilizer:Stabilizer_MX_6.25u, F.Cu at (217.3, 201.6)
- added REF**: Stabilizer_MX_2.00u, ScottoKeebs_Stabilizer:Stabilizer_MX_2.00u, F.Cu at (341.1, 182.6)
- added REF**: Stabilizer_MX_2.00u, ScottoKeebs_Stabilizer:Stabilizer_MX_2.00u, F.Cu at (345.9, 163.5)
- S4, S7: footprint ScottoKeebs_MX:MX_PCB_1.00u -> ScottoKeebs_MX:MX_PCB_1.50u
- S42: footprint ScottoKeebs_MX:MX_PCB_1.00u -> ScottoKeebs_MX:MX_PCB_2.25u
- S43: footprint ScottoKeebs_MX:MX_PCB_1.00u -> ScottoKeebs_MX:MX_PCB_2.00u
- S44, S46, S48, S52, S54, S58, S72: footprint ScottoKeebs_MX:MX_PCB_1.00u -> ScottoKeebs_MX:MX_PCB_1.25u
- S50: footprint ScottoKeebs_MX:MX_PCB_1.00u -> ScottoKeebs_MX:MX_PCB_6.25u
- S67: footprint ScottoKeebs_MX:MX_PCB_1.00u -> ScottoKeebs_MX:MX_PCB_2.75u
- S71: footprint ScottoKeebs_MX:MX_PCB_1.00u -> ScottoKeebs_MX:MX_PCB_1.75u
- moved D48 14.3 mm to (157.8, 204.2)
- moved SW4 12.4 mm to (199.9, 202.3)
- moved SW3 12.2 mm to (199.9, 197.5)
- moved J6 12.0 mm to (185.1, 201.6)
- moved S48 11.9 mm to (145.9, 201.6)
- moved D46 9.53 mm to (133.9, 204.0)
- moved S52 7.14 mm to (288.7, 201.6)
- moved S46 7.14 mm to (122.0, 201.6)
- moved D38 4.76 mm to (324.4, 146.9)
- moved D39 4.76 mm to (324.4, 165.9)
- moved D52 4.76 mm to (300.6, 204.0)
- moved S29 4.76 mm to (276.8, 144.5)
- moved S30 4.76 mm to (276.8, 163.5)
- moved D17 4.76 mm to (210.1, 146.9)
- moved D18 4.76 mm to (210.1, 165.9)
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Routing:
- net col4: track 304.6 -> 229.9 mm, vias 0 -> 1
- net col5: track 323.9 -> 281.3 mm
- net col6: track 366.1 -> 338.6 mm, vias 1 -> 0
- net row2: track 444.9 -> 461.6 mm, vias 1 -> 0
- net col0: track 224.0 -> 238.6 mm
- net col12: track 329.2 -> 316.3 mm
- net /D4-: track 222.7 -> 235.4 mm
- net col9: track 375.0 -> 362.3 mm
- net col13: track 308.3 -> 295.7 mm
- net col10: track 356.4 -> 343.8 mm
- net col8: track 387.9 -> 375.5 mm
- net /D4+: track 191.6 -> 203.7 mm
- net col2: track 173.2 -> 183.4 mm
- net row3: track 275.0 -> 285.0 mm
- net col1: track 217.6 -> 226.1 mm
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