File: pcb/pcb.kicad_sch (KiCad schematic)
At the start: 165 parts, among them J1 USB_C_Receptacle_USB2.0, J2 USB_C_Receptacle_USB2.0, J4 USB_C_Receptacle_USB2.0, J5 USB_C_Receptacle_USB2.0, SW1 SW_Push, U1 SL2.1A, U2 NCP1117-3.3_SOT223, U3 W25Q128JVS, U4 RP2040, Y1 ABM8-272-T3

Commit message: Redesign
Parts:
- added H1, H2, H3, H4, H5, H6: MountingHole, MountingHole:MountingHole_2.1mm, symbol Mechanical:MountingHole
- S1, S10, S11, S12, S13, S14, S15, S16, S17, S18, S19, S2, S20, S21, S22, S23, S24, S25, S26, S27, S28, S29, S3, S30, S31, S32, S33, S37, S38, S39, S40, S41, S45, S47, S49, S5, S51, S53, S55, S56, S57, S59, S6, S61, S63, S8, S9: footprint ScottoKeebs_MX:MX_PCB_1.00u -> Switch_Keyboard_Hotswap_Kailh:SW_Hotswap_Kailh_MX_1.00u
- S4, S7: footprint ScottoKeebs_MX:MX_PCB_1.50u -> Switch_Keyboard_Hotswap_Kailh:SW_Hotswap_Kailh_MX_1.00u
- S42: footprint ScottoKeebs_MX:MX_PCB_2.25u -> Switch_Keyboard_Hotswap_Kailh:SW_Hotswap_Kailh_MX_2.25u
- S43: footprint ScottoKeebs_MX:MX_PCB_2.00u -> Switch_Keyboard_Hotswap_Kailh:SW_Hotswap_Kailh_MX_2.00u
- S44, S46, S48, S52, S54, S58, S72: footprint ScottoKeebs_MX:MX_PCB_1.25u -> Switch_Keyboard_Hotswap_Kailh:SW_Hotswap_Kailh_MX_1.25u
- S50: footprint ScottoKeebs_MX:MX_PCB_6.25u -> Switch_Keyboard_Hotswap_Kailh:SW_Hotswap_Kailh_MX_6.25u
- S67: footprint ScottoKeebs_MX:MX_PCB_2.75u -> Switch_Keyboard_Hotswap_Kailh:SW_Hotswap_Kailh_MX_2.75u
- S71: footprint ScottoKeebs_MX:MX_PCB_1.75u -> Switch_Keyboard_Hotswap_Kailh:SW_Hotswap_Kailh_MX_1.75u

Commit message: Fixed Traces
Parts:
- U3: footprint Package_SO:SOIC-8_5.23x5.23mm_P1.27mm -> Package_SO:SOIC-8_5.3x5.3mm_P1.27mm
